File: eagle_schematics/current-sense.sch (EAGLE design)
At the start: 19 parts, among them IC1 MCP601P

Commit message: mais esquemáticos
Parts:
- removed BUFFER: MCP601P, linear:MCP601P
- added C2: (no value), rcl:C-EU075-032X103
- added IC2: MCP602P, linear:MCP602P
- IC1: value MCP601P -> MCP602P; device linear:MCP601P -> linear:MCP602P
- R1, R2: value 330 -> 470
- R3: value 6k8 -> 1k
- R4: value 4k7 -> 1k
- R5: value 6k8 -> 8k2
- R6: value 5k6 -> 3k3
- R8: value 180 -> 100
- R9: value 3k9 -> 180
Connections:
- removed net N$16: C1.2, D1.C, IC1.V-, R7.1, R8.2, TL431.A
- removed net N$5: 557-1.B, IC1.OUT
- new net N$3: 557-1.B, IC2A.OUT
- new net N$4: 557-2.E, C1.1, C2.1, IC2A.-IN, R2.2, R6.2, TL431.C
- net AGND: now also IC1P.V-; no longer BUFFER.V-
- net N$1: now also C1.2, C2.2, D1.C, IC2P.V-, R7.1, R8.2, TL431.A; no longer 557-2.E, C1.1, IC1.-IN, R2.2, R6.2, TL431.C
- net N$2: now also IC2A.+IN; no longer IC1.+IN
- net N$9: now also IC1A.+IN; no longer BUFFER.+IN
- net OUT: now also IC1A.-IN, IC1A.OUT; no longer BUFFER.-IN, BUFFER.OUT
- net SN: now also IC2P.V+; no longer IC1.V+
- net VCC: now also IC1P.V+; no longer BUFFER.V+
Other:
- note added: "Current Sink"
- note added: "OutPut PIC32 ADC"
- note added: "Sensing Resistor"
- note added: "Vblue"
- note added: "Voltage Reference"
- note added: "Vred"
- note removed: "OUT"
- note removed: "SN"
- note removed: "SP"
- moved on the sheet: 557-BIAS, D1, R4, R8, R9

Commit message: atualizacao de modelos 3D e esquematicos
Connections:
- net N$4: no longer C1.1, C2.1, R6.2, TL431.C
- net SN: now also C1.1, C2.1, R6.2, TL431.C
Other:
- moved on the sheet: IC2B
