File: eagle_schematics/pwmControl.brd (EAGLE design)
At the start: 120.6 x 72.1 mm, 18 parts, among them IC1 TL081P, IC2 MCP602P, Q1 VN66AF, Q2 BD139

Commit message: atualizacao de modelos 3D e esquematicos
Parts:
- moved D3 215.3 mm to (80.0, 74.9), turned to 90 degrees
- moved R9 212.1 mm to (85.1, 86.4), turned to 180 degrees
- moved R8 196.1 mm to (80.0, 87.6), turned to 90 degrees
- moved J1 148.2 mm to (52.1, 74.9), turned to 270 degrees
- moved D2 135.7 mm to (69.8, 67.3)
- moved IC2 126.1 mm to (66.0, 78.7)
- moved R7 112.4 mm to (83.8, 67.3), turned to 180 degrees
- moved R6 87.1 mm to (61.0, 71.1), turned to 180 degrees
- moved R5 13.3 mm to (43.2, 85.1), turned to 90 degrees
Connections:
- net N$1 renamed OUTFAN
- net N$11 renamed PWMVOLTAGE
- net N$14 renamed VOUTRED
- net N$4 renamed PWMFAN
- net N$8 renamed 2N3055BASE
- net N$9 renamed 2N3055COL
- removed net N$12: IC2.1, IC2.2, J1.10
- removed net N$16: J1.8, R7.1
- removed net N$17: J1.9, R9.1
- new net VINBAT: J1.1, R7.1
- new net VINRED: J1.8, R9.1
- new net VOUTBATT: IC2.1, IC2.2, J1.9
- net VCC: now also J1.10; no longer J1.1
Routing:
- net VCC: track 16.1 -> 137.9 mm
- net VINRED: track 0.00 -> 81.4 mm
- net VINBAT: track 0.00 -> 47.5 mm
- net VOUTRED: track 0.00 -> 25.8 mm
- net VOUTBATT: track 0.00 -> 21.6 mm
- net N$10: track 0.00 -> 19.4 mm
- net N$13: track 0.00 -> 17.8 mm
- net PWMVOLTAGE: track 0.00 -> 14.2 mm
- net 2N3055BASE: track 58.3 -> 47.9 mm
- net OUTFAN: track 58.5 -> 49.0 mm
- net 2N3055COL: track 36.5 -> 44.3 mm
- net N$6: track 41.9 -> 40.0 mm
- net PWMFAN: track 73.2 -> 74.5 mm
Other:
- board size 120.6 x 72.1 mm -> 87.6 x 60.6 mm
