File: eagle_schematics/pwmControl.sch (EAGLE design)
At the start: 18 parts, among them IC1 TL081P, IC2 MCP602P, Q1 VN66AF, Q2 BD139

Commit message: atualizacao de modelos 3D e esquematicos
Connections:
- net N$1 renamed OUTFAN
- net N$11 renamed PWMVOLTAGE
- net N$14 renamed VOUTRED
- net N$4 renamed PWMFAN
- net N$8 renamed 2N3055BASE
- net N$9 renamed 2N3055COL
- removed net N$12: IC2A.-IN, IC2A.OUT, J1.10
- removed net N$16: J1.8, R7.1
- removed net N$17: J1.9, R9.1
- new net VINBAT: J1.1, R7.1
- new net VINRED: J1.8, R9.1
- new net VOUTBATT: IC2A.-IN, IC2A.OUT, J1.9
- net VCC: now also J1.10; no longer J1.1
Other:
- moved on the sheet: D2, D3, IC2A, IC2B, R6, R7, R8, R9
